File: comp_and_pwr_pcb.kicad_pcb (KiCad board)
At the start: 4 copper layers, 50 x 88.5 mm, 145 parts, among them IC1 TPS5430MDDAREP, IC3 LTC4415EDHC#TRPBF, IC4 TPS259531DSGR, IC5 BMP388, IC6 W25Q32JVSSIQ, J1 USB4216-03-A, J10 Conn_01x02, J11 Conn_Coaxial, J12 Conn_Coaxial, J2 BATTERY_CONN, J3 SWD_CONN, J4 SERVO_CONN_01, J5 SERVO_CONN_02, J6 DM3AT-SF-PEJM5, J7 CAMERA_CONN_01, J8 CAMERA_CONN_02, J9 Conn_01x02, Q1 2N3904, Q2 BSS138, Q3 BSS138, Q4 BC847B, Q5 BC847B, Q6 DMP3013SFV, Q8 DMP3013SFV, SW1 SW_Push, SW2 SW_Push, U1 RP2040, U2 MAX-M10S, U3 MP2307DN-LF-Z, U4 LSM6DSO, Y1 ABMM2-12.000MHZ-D1-T

Commit message: hotswapchip fixed
Parts:
- removed C10: 4.7uF, Capacitor_SMD:C_0402_1005Metric
- removed C26, C32: 100nF, Capacitor_SMD:C_0402_1005Metric
- removed C27, C31: 10uF, Capacitor_SMD:C_0402_1005Metric
- removed D3: D_TVS, Diode_SMD:D_SOD-523
- removed IC3: LTC4415EDHC#TRPBF, Package_DFN_QFN:DFN-18-1EP_3x5mm_P0.5mm_EP1.66x4.4mm
- removed JP2: SolderJumper_3_Open, Jumper:SolderJumper-3_P1.3mm_Open_Pad1.0x1.5mm
- removed R10, R9: 124, Resistor_SMD:R_0402_1005Metric
- removed R11: 100k, Resistor_SMD:R_0402_1005Metric
- removed R21: 21.5k, Resistor_SMD:R_0402_1005Metric
- removed the R24 at (140.8, 147.3)
- removed R9: 47k, Resistor_SMD:R_0402_1005Metric
- removed U4: LSM6DSO, LSM6DSO:LGA14L
- added C14: 10uF, Capacitor_SMD:C_0402_1005Metric, F.Cu at (139.0, 152.5)
- added C21: 100nF, Capacitor_SMD:C_0402_1005Metric, F.Cu at (135.0, 146.0)
- added C22: 10uF, Capacitor_SMD:C_0402_1005Metric, F.Cu at (135.0, 144.5)
- added C25: 100nF, Capacitor_SMD:C_0402_1005Metric, F.Cu at (139.0, 153.5)
- added IC2: ICM-42688-P, ICM-42688-P:IIM42352, F.Cu at (135.0, 149.5)
- added JP4: SolderJumper_3_Open, Jumper:SolderJumper-3_P1.3mm_Open_Pad1.0x1.5mm, F.Cu at (135.0, 141.5)
- added Q10: PMV28XPEAR, Package_TO_SOT_SMD:SOT-23, F.Cu at (116.5, 136.0)
- added R28: 1k, Resistor_SMD:R_0402_1005Metric, F.Cu at (106.0, 156.0)
- added R31: 100k, Resistor_SMD:R_0402_1005Metric, F.Cu at (106.0, 153.4)
- C11, C13, C2, C24, C39: footprint Capacitor_SMD:C_1206_3216Metric -> Capacitor_SMD:C_0402_1005Metric
- C23: footprint Capacitor_SMD:C_0603_1608Metric -> Capacitor_SMD:C_0805_2012Metric
- C36: footprint Capacitor_SMD:C_1206_3216Metric -> E22-400M22S:CP_EIA-7343-43_Vishay-E_Pad2.25x2.55mm_HandSolder
- C42, C6, C9: footprint Capacitor_SMD:C_0603_1608Metric -> Capacitor_SMD:C_0402_1005Metric
- D1, D2: footprint Diode_SMD:D_SOD-523 -> Package_TO_SOT_SMD:SOT-23
- Q6, Q8: value DMP3013SFV -> PMV28XPEAR; footprint Package_SON:Diodes_PowerDI3333-8 -> Package_TO_SOT_SMD:SOT-23
- moved Q6 20.5 mm to (109.3, 155.2)
- moved D5 12.7 mm to (140.0, 104.8)
- moved C36 3.90 mm to (119.7, 93.3), turned to -90 degrees
- moved D2 1.82 mm to (130.4, 125.6), turned to 180 degrees
- moved D1 1.28 mm to (133.8, 116.5)
- moved C23 1.07 mm to (107.8, 147.8), turned to 0 degrees
- moved C11 0.55 mm to (105.3, 148.6), turned to -90 degrees
- moved J4 0.46 mm to (140.5, 109.0)
- moved R26 0.15 mm to (108.7, 149.9)
Connections:
- net RF_NET renamed Net-(E22-400M22S1-ANT)
- C8 pad 2: /5V_BATT -> 5V_BATT
- C9 pad 2: /5V_BATT -> 5V_BATT
- L1 pad 2: /5V_BATT -> 5V_BATT
- Q6 pad 1: +BATT -> Net-(Q6-G)
- Q6 pad 2: +BATT -> 5V_BATT
- Q6 pad 3: +BATT -> +5V
- Q8 pad 1: +BATT -> Net-(Q8-G)
- Q8 pad 3: +BATT -> Net-(J10-Pin_1)
- R62 pad 1: Net-(Q6-G) -> Net-(Q10-G)
- R7 pad 2: /5V_BATT -> 5V_BATT
Routing:
- net /USB_DM: track 51.4 -> 11.8 mm, vias 5 -> 2
- net /USB_DP: track 44.0 -> 12.2 mm, vias 3 -> 2
- net /5V_BATT: track 24.2 -> 0.00 mm
- net 5V_BATT: track 0.00 -> 20.5 mm
- net Net-(IC3-EN1): track 18.9 -> 0.00 mm, vias 2 -> 0
- net /5V_USB: track 90.6 -> 78.8 mm, vias 4 -> 3
- net Net-(D5-A2): track 11.7 -> 22.2 mm
- net Net-(IC3-CLIM2): track 9.37 -> 0.00 mm, vias 2 -> 0
- net +5V: track 76.6 -> 67.3 mm, vias 6 -> 5
- net Net-(IC3-CLIM1): track 8.94 -> 0.00 mm, vias 2 -> 0
- net Net-(IC2-AP_SDO_/_AP_AD0): track 0.00 -> 7.78 mm
- net Net-(JP2-C): track 7.17 -> 0.00 mm, vias 2 -> 0
- net Net-(Q6-G): track 11.0 -> 4.14 mm
- net GND: track 259.3 -> 266.1 mm, vias 61 -> 58
- net Net-(Q10-G): track 0.00 -> 4.86 mm, vias 0 -> 2
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Other:
- board text removed: "2025"
- board text removed: "BATT"
- board text removed: "CAM_01"
- board text removed: "CAM_02"
- board text removed: "GPS"
- board text removed: "LoRa"
- board text removed: "PYRO_1"
- board text removed: "PYRO_2"
- board text removed: "RTU HPR"
- board text removed: "SERVO"
