File: comp_and_pwr_pcb.kicad_sch (KiCad schematic)
At the start: 143 parts, among them IC1 TPS5430MDDAREP, IC3 LTC4415EDHC#TRPBF, IC4 TPS259531DSGR, IC5 BMP388, IC6 W25Q32JVSSIQ, J1 USB4216-03-A, J10 Conn_01x02, J11 Conn_Coaxial, J12 Conn_Coaxial, J2 BATTERY_CONN, J3 SWD_CONN, J4 SERVO_CONN_01, J5 SERVO_CONN_02, J6 DM3AT-SF-PEJM5, J7 CAMERA_CONN_01, J8 CAMERA_CONN_02, J9 Conn_01x02, Q1 2N3904, Q2 BSS138, Q3 BSS138, Q4 BC847B, Q5 BC847B, Q6 DMP3013SFV, Q8 DMP3013SFV, SW1 SW_Push, SW2 SW_Push, U1 RP2040, U2 MAX-M10S, U3 MP2307DN-LF-Z, U4 LSM6DSO, Y1 ABMM2-12.000MHZ-D1-T

Commit message: hotswapchip fixed
Parts:
- removed C26, C32: 100nF, Capacitor_SMD:C_0402_1005Metric, symbol Device:C_Small
- removed C27, C31: 10uF, Capacitor_SMD:C_0402_1005Metric, symbol Device:C_Small
- removed D3: D_TVS, Diode_SMD:D_SOD-523, symbol Device:D_TVS
- removed JP2: SolderJumper_3_Open, Jumper:SolderJumper-3_P1.3mm_Open_Pad1.0x1.5mm, symbol Jumper:SolderJumper_3_Open
- removed Q6, Q8: DMP3013SFV, Package_SON:Diodes_PowerDI3333-8, symbol Transistor_FET:DMP3013SFV
- removed U4: LSM6DSO, LSM6DSO:LGA14L, symbol LSM6DSO:LSM6DSO
- added C14, C22: 10uF, Capacitor_SMD:C_0402_1005Metric, symbol Device:C_Small
- added C21, C25: 100nF, Capacitor_SMD:C_0402_1005Metric, symbol Device:C_Small
- added IC2: ICM-42688-P, ICM-42688-P:IIM42352, symbol ICM-42688-P:ICM-42688-P
- added JP4: SolderJumper_3_Open, Jumper:SolderJumper-3_P1.3mm_Open_Pad1.0x1.5mm, symbol Jumper:SolderJumper_3_Open
- added Q10, Q6, Q8: PMV28XPEAR, Package_TO_SOT_SMD:SOT-23, symbol PMV28XPEAR:PMV28XPEAR
- added R28: 1k, Resistor_SMD:R_0402_1005Metric, symbol Device:R
- added R31: 100k, Resistor_SMD:R_0402_1005Metric, symbol Device:R
- BZ1: MPN CPT-9019S-SMT-TR -> (none); Manufacturer Same Sky -> (none)
- C1, C3: MPN C0402C300F5GAC -> (none); Manufacturer KEMET -> (none)
- C10: MPN C0805C475K8PACTU -> (none); Manufacturer KEMET -> (none); now not fitted
- C11, C13, C2, C24, C39: footprint Capacitor_SMD:C_1206_3216Metric -> Capacitor_SMD:C_0402_1005Metric; MPN C0402C106M9PACTU -> (none); Manufacturer KEMET -> (none)
- C12, C16, C17, C18, C4: MPN C0402C104K4RAC7411 -> (none); Manufacturer Yageo -> (none)
- C15, C19: MPN C0402C105K8PACTU -> (none); Manufacturer KEMET -> (none)
- C20, C28, C29, C34, C38, C40, C41, C43, C5, C52, C8: MPN C0402C104K4RAC7411 -> (none); Manufacturer KEMET -> (none)
- C23: footprint Capacitor_SMD:C_0603_1608Metric -> Capacitor_SMD:C_0805_2012Metric; MPN C0805C475K8PACTU -> (none); Manufacturer KEMET -> (none)
- C30: MPN 6TPF470MFH -> (none); Manufacturer Panasonic -> (none)
- C35: MPN C0402C106M9PACTU -> (none); Manufacturer KEMET -> (none)
- C36: footprint Capacitor_SMD:C_1206_3216Metric -> E22-400M22S:CP_EIA-7343-43_Vishay-E_Pad2.25x2.55mm_HandSolder; MPN T495X476K020AHE150 -> (none); Manufacturer KEMET -> (none)
- C42, C6, C9: footprint Capacitor_SMD:C_0603_1608Metric -> Capacitor_SMD:C_0402_1005Metric; MPN C0402C106M9PACTU -> (none); Manufacturer KEMET -> (none)
- C51: MPN KEMET -> (none); Manufacturer C0402C104K4RAC7411 -> (none)
- C7: MPN GRM1555C1H101FA01D -> (none); Manufacturer Murata Electronics -> (none)
- D1, D2: footprint Diode_SMD:D_SOD-523 -> Package_TO_SOT_SMD:SOT-23; MPN ESD5Z5.0T1G -> (none); Manufacturer onsemi -> (none)
- D4: MPN SZSMF6L5.0AT3G -> (none); Manufacturer Littelfuse -> (none)
- D5: renamed from BAS70S-AU_R1_000A1; MPN BAS70S-AU_R1_000A1 -> (none); Manufacturer Panjit -> (none)
- F1: MPN 0ABA-1000-TN -> (none); Manufacturer Bel Fuse -> (none)
- F2: MPN 2016L200PR -> (none); Manufacturer Littelfuse -> (none)
- IC1: MPN TPS5430MDDAREP -> (none); Manufacturer Texas Instruments -> (none)
- IC3: MPN LTC4415EDHC#TRPBF -> (none); Manufacturer Analog Devices -> (none); now not fitted
- IC4: MPN TPS259531DSGR -> (none); Manufacturer Texas Instruments -> (none)
- IC5: MPN BMP388 -> (none); Manufacturer Bosch -> (none)
- IC6: MPN W25Q32JVSSIQ -> (none); Manufacturer Winbond -> (none)
- J1: MPN USB4216-03-A -> (none); Manufacturer GCT -> (none)
- J10, J2, J7, J8, J9: MPN 284514-2 -> (none); Manufacturer TE Connectivity -> (none)
- J11, J12: MPN 73251-2200 -> (none); Manufacturer Molex -> (none)
- J3: MPN M20-9990546 -> (none); Manufacturer Harwin -> (none)
- J4, J5: MPN 90131-0763 -> (none); Manufacturer Molex -> (none)
- J6: MPN DM3AT-SF-PEJM5 -> (none); Manufacturer Hirose Connector -> (none)
- L1, L2: MPN 74437349033 -> (none); Manufacturer Wurth Elektronik -> (none)
- Q1: MPN MMBT3904 -> (none); Manufacturer Diotec Semiconductor -> (none)
- Q2, Q3: MPN BSS138 -> (none); Manufacturer onsemi / Fairchild -> (none)
- Q4, Q5: MPN BC847B -> (none); Manufacturer Diotec Semiconductor -> (none)
- R1, R14, R20: MPN RC0402FR‑071KL -> (none); Manufacturer Yageo -> (none)
- R10, R9: MPN RC0402FR-07124RL -> (none); Manufacturer Yageo -> (none); now not fitted
- R11: MPN RC0402FR-07100KL -> (none); Manufacturer Yageo -> (none); now not fitted
- R12, R13: MPN RC0402JR-7D33RL -> (none); Manufacturer Yageo -> (none)
- R15, R16, R29, R30, R39, R40, R45, R59, R61, R7: MPN RC0402FR-0710KL -> (none); Manufacturer Yageo -> (none)
- R17: MPN RC0402FR-075K6L -> (none); Manufacturer Yageo -> (none)
- R19, R22, R23: MPN RC1206FR-07100RL -> (none); Manufacturer Yageo -> (none)
- R2, R3: MPN RC0402FR-075K1L -> (none); Manufacturer Yageo -> (none)
- R21: MPN RC0402FR-0721K5L -> (none); Manufacturer Yageo -> (none); now not fitted
- R24: MPN RC0402FR-075K76L -> (none); Manufacturer Yageo -> (none)
- R25, R57, R6, R63: MPN RC0402FR-07100KL -> (none); Manufacturer Yageo -> (none)
- R26: MPN RC0402FR-076K8L -> (none); Manufacturer Yageo -> (none)
- R27: MPN RC0402FR-0726K1L -> (none); Manufacturer Yageo -> (none)
- R32: MPN RC0603FR-0715K8L -> (none); Manufacturer Yageo -> (none)
- R35, R36, R37, R38: MPN RC0402FR-07100RL -> (none); Manufacturer Yageo -> (none)
- R4, R5: MPN RC0402FR-0722RL -> (none); Manufacturer Yageo -> (none)
- R41, R42: MPN RC0402FR-07220R -> (none); Manufacturer Yageo -> (none)
- R43, R44: MPN RC0402FR-074K7L -> (none); Manufacturer Yageo -> (none)
- R48: MPN RC0402FR-07220RL -> (none); Manufacturer Yageo -> (none)
- R54: MPN RC0402FR-071KL -> (none); Manufacturer Yageo -> (none)
- R58, R62: MPN RC0402FR-0747RL -> (none); Manufacturer Yageo -> (none)
- R60, R64: MPN RC0402FR-073K3L -> (none); Manufacturer Yageo -> (none)
- R8: MPN RC0402FR-073R24L -> (none); Manufacturer Yageo -> (none)
- STATUS1: MPN COM-24837 -> (none); Manufacturer SparkFun -> (none)
- SW1, SW2: MPN PTS645SM43SMTR92 -> (none); Manufacturer C&K -> (none)
- TX1, TX2, TX3, TX4: MPN XL-1608UBC-04 -> (none); Manufacturer XINGLIGHT -> (none)
- U1: MPN RP2040 -> (none); Manufacturer Raspberry Pi -> (none)
- U2: MPN MAX-M10S-00B -> (none); Manufacturer u-blox -> (none)
- U3: MPN MP2307DN-LF-Z -> (none); Manufacturer Monolithic Power Systems (MPS) -> (none)
- Y1: MPN ABMM2-12.000MHZ-D1-T -> (none); Manufacturer ABRACON -> (none)
Connections:
- net +3.3V: now also C14.2, C21.2, C22.2, C25.1, IC2.12 (AP_CS), IC2.5 (VDDIO), IC2.8 (VDD), JP4.1 (A)
- net +5V: now also Q6.3 (D)
- net +BATT: now also Q10.2 (S), Q8.2 (S)
- net 5V_BATT: now also Q6.2 (S)
- net 5V_USB: now also R28.1
- net GND: now also C14.1, C21.1, C22.1, C25.2, IC2.6 (GND), JP4.3 (B), R31.1
- net I2C_SCL: now also IC2.13 (AP_SCL_/_AP_SCLK)
- net I2C_SDA: now also IC2.14 (AP_SDA_/_AP_SDIO_/_AP_SDI)
- net at J9.1 (Pin_1), R64.1: now also Q10.3 (D)
- net at R58.1: now also Q8.1 (G)
- net at J10.1 (Pin_1), R60.1: now also Q8.3 (D)
- net at R62.1: now also Q10.1 (G)
- new net: Q6.1 (G), R28.2, R31.2
- new net: IC2.1 (AP_SDO_/_AP_AD0), JP4.2 (C)
- no-connect marks 40 -> 41
Other:
- moved on the sheet: R17, R25
