File: ARC_PFC.kicad_sch (KiCad schematic)
At the start: 145 parts, among them IC1 TPS5430MDDAREP, IC2 ICM-42688-P, IC3 LTC4415EDHC#TRPBF, IC4 TPS259531DSGR, IC5 BMP388, IC6 W25Q32JVSSIQ, J1 USB4216-03-A, J10 Conn_01x02, J11 Conn_Coaxial, J12 Conn_Coaxial, J2 BATTERY_CONN, J3 SWD_CONN, J4 SERVO_CONN_01, J5 SERVO_CONN_02, J6 DM3AT-SF-PEJM5, J7 CAMERA_CONN_01, J8 CAMERA_CONN_02, J9 Conn_01x02, Q1 2N3904, Q10 PMV28XPEAR, Q2 BSS138, Q3 BSS138, Q4 BC847B, Q5 BC847B, Q6 PMV28XPEAR, Q8 PMV28XPEAR, SW1 SW_Push, SW2 SW_Push, U1 RP2040, U2 MAX-M10S, U3 MP2307DN-LF-Z, Y1 ABMM2-12.000MHZ-D1-T

Commit message: naming fixed
Parts:
- removed C14, C22: 10uF, Capacitor_SMD:C_0402_1005Metric, symbol Device:C_Small
- removed C21, C25: 100nF, Capacitor_SMD:C_0402_1005Metric, symbol Device:C_Small
- removed IC2: ICM-42688-P, ICM-42688-P:IIM42352, symbol ICM-42688-P:ICM-42688-P
- removed JP4: SolderJumper_3_Open, Jumper:SolderJumper-3_P1.3mm_Open_Pad1.0x1.5mm, symbol Jumper:SolderJumper_3_Open
- removed Q10, Q6, Q8: PMV28XPEAR, Package_TO_SOT_SMD:SOT-23, symbol PMV28XPEAR:PMV28XPEAR
- removed R28: 1k, Resistor_SMD:R_0402_1005Metric, symbol Device:R
- removed R31: 100k, Resistor_SMD:R_0402_1005Metric, symbol Device:R
- added C26, C32: 100nF, Capacitor_SMD:C_0402_1005Metric, symbol Device:C_Small
- added C27, C31: 10uF, Capacitor_SMD:C_0402_1005Metric, symbol Device:C_Small
- added D3: D_TVS, Diode_SMD:D_SOD-523, symbol Device:D_TVS
- added JP2: SolderJumper_3_Open, Jumper:SolderJumper-3_P1.3mm_Open_Pad1.0x1.5mm, symbol Jumper:SolderJumper_3_Open
- added Q6, Q8: DMP3013SFV, Package_SON:Diodes_PowerDI3333-8, symbol Transistor_FET:DMP3013SFV
- added U4: LSM6DS0, LSM6DSO:LGA14L, symbol LSM6DSO:LSM6DSO
- BAS70S-AU_R1_000A1: renamed from D5; MPN (none) -> BAS70S-AU_R1_000A1; Manufacturer (none) -> Panjit
- BZ1: MPN (none) -> CPT-9019S-SMT-TR; Manufacturer (none) -> Same Sky
- C1, C3: MPN (none) -> C0402C300F5GAC; Manufacturer (none) -> KEMET
- C10: MPN (none) -> C0805C475K8PACTU; Manufacturer (none) -> KEMET; now fitted
- C11, C13, C2, C24, C39: footprint Capacitor_SMD:C_0402_1005Metric -> Capacitor_SMD:C_1206_3216Metric; MPN (none) -> C0402C106M9PACTU; Manufacturer (none) -> KEMET
- C12, C16, C17, C18, C4: MPN (none) -> C0402C104K4RAC7411; Manufacturer (none) -> Yageo
- C15, C19: MPN (none) -> C0402C105K8PACTU; Manufacturer (none) -> KEMET
- C20, C28, C29, C34, C38, C40, C41, C43, C5, C52, C8: MPN (none) -> C0402C104K4RAC7411; Manufacturer (none) -> KEMET
- C23: footprint Capacitor_SMD:C_0805_2012Metric -> Capacitor_SMD:C_0603_1608Metric; MPN (none) -> C0805C475K8PACTU; Manufacturer (none) -> KEMET
- C30: MPN (none) -> 6TPF470MFH; Manufacturer (none) -> Panasonic
- C35: MPN (none) -> C0402C106M9PACTU; Manufacturer (none) -> KEMET
- C36: footprint E22-400M22S:CP_EIA-7343-43_Vishay-E_Pad2.25x2.55mm_HandSolder -> Capacitor_SMD:C_1206_3216Metric; MPN (none) -> T495X476K020AHE150; Manufacturer (none) -> KEMET
- C42, C6, C9: footprint Capacitor_SMD:C_0402_1005Metric -> Capacitor_SMD:C_0603_1608Metric; MPN (none) -> C0402C106M9PACTU; Manufacturer (none) -> KEMET
- C51: MPN (none) -> KEMET; Manufacturer (none) -> C0402C104K4RAC7411
- C7: MPN (none) -> GRM1555C1H101FA01D; Manufacturer (none) -> Murata Electronics
- D1, D2: footprint Package_TO_SOT_SMD:SOT-23 -> Diode_SMD:D_SOD-523; MPN (none) -> ESD5Z5.0T1G; Manufacturer (none) -> onsemi
- D4: MPN (none) -> SZSMF6L5.0AT3G; Manufacturer (none) -> Littelfuse
- E22-400M22S1: value ~ -> (none)
- F1: MPN (none) -> 0ABA-1000-TN; Manufacturer (none) -> Bel Fuse
- F2: MPN (none) -> 2016L200PR; Manufacturer (none) -> Littelfuse
- IC1: MPN (none) -> TPS5430MDDAREP; Manufacturer (none) -> Texas Instruments
- IC3: MPN (none) -> LTC4415EDHC#TRPBF; Manufacturer (none) -> Analog Devices; now fitted
- IC4: MPN (none) -> TPS259531DSGR; Manufacturer (none) -> Texas Instruments
- IC5: MPN (none) -> BMP388; Manufacturer (none) -> Bosch
- IC6: MPN (none) -> W25Q32JVSSIQ; Manufacturer (none) -> Winbond
- J1: MPN (none) -> USB4216-03-A; Manufacturer (none) -> GCT
- J10, J2, J7, J8, J9: MPN (none) -> 284514-2; Manufacturer (none) -> TE Connectivity
- J11, J12: MPN (none) -> 73251-2200; Manufacturer (none) -> Molex
- J3: MPN (none) -> M20-9990546; Manufacturer (none) -> Harwin
- J4, J5: MPN (none) -> 90131-0763; Manufacturer (none) -> Molex
- J6: MPN (none) -> DM3AT-SF-PEJM5; Manufacturer (none) -> Hirose Connector
- L1, L2: MPN (none) -> 74437349033; Manufacturer (none) -> Wurth Elektronik
- Q1: MPN (none) -> MMBT3904; Manufacturer (none) -> Diotec Semiconductor
- Q2, Q3: MPN (none) -> BSS138; Manufacturer (none) -> onsemi / Fairchild
- Q4, Q5: MPN (none) -> BC847B; Manufacturer (none) -> Diotec Semiconductor
- R1, R14, R20: MPN (none) -> RC0402FR‑071KL; Manufacturer (none) -> Yageo
- R10, R9: MPN (none) -> RC0402FR-07124RL; Manufacturer (none) -> Yageo; now fitted
- R11: MPN (none) -> RC0402FR-07100KL; Manufacturer (none) -> Yageo; now fitted
- R12, R13: MPN (none) -> RC0402JR-7D33RL; Manufacturer (none) -> Yageo
- R15, R16, R29, R30, R39, R40, R45, R59, R61, R7: MPN (none) -> RC0402FR-0710KL; Manufacturer (none) -> Yageo
- R17: MPN (none) -> RC0402FR-075K6L; Manufacturer (none) -> Yageo
- R19, R22, R23: MPN (none) -> RC1206FR-07100RL; Manufacturer (none) -> Yageo
- R2, R3: MPN (none) -> RC0402FR-075K1L; Manufacturer (none) -> Yageo
- R21: MPN (none) -> RC0402FR-0721K5L; Manufacturer (none) -> Yageo; now fitted
- R24: MPN (none) -> RC0402FR-075K76L; Manufacturer (none) -> Yageo
- R25, R57, R6, R63: MPN (none) -> RC0402FR-07100KL; Manufacturer (none) -> Yageo
- R26: MPN (none) -> RC0402FR-076K8L; Manufacturer (none) -> Yageo
- R27: MPN (none) -> RC0402FR-0726K1L; Manufacturer (none) -> Yageo
- R32: MPN (none) -> RC0603FR-0715K8L; Manufacturer (none) -> Yageo
- R35, R36, R37, R38: MPN (none) -> RC0402FR-07100RL; Manufacturer (none) -> Yageo
- R4, R5: MPN (none) -> RC0402FR-0722RL; Manufacturer (none) -> Yageo
- R41, R42: MPN (none) -> RC0402FR-07220R; Manufacturer (none) -> Yageo
- R43, R44: MPN (none) -> RC0402FR-074K7L; Manufacturer (none) -> Yageo
- R48: MPN (none) -> RC0402FR-07220RL; Manufacturer (none) -> Yageo
- R54: MPN (none) -> RC0402FR-071KL; Manufacturer (none) -> Yageo
- R58, R62: MPN (none) -> RC0402FR-0747RL; Manufacturer (none) -> Yageo
- R60, R64: MPN (none) -> RC0402FR-073K3L; Manufacturer (none) -> Yageo
- R8: MPN (none) -> RC0402FR-073R24L; Manufacturer (none) -> Yageo
- STATUS1: MPN (none) -> COM-24837; Manufacturer (none) -> SparkFun
- SW1, SW2: MPN (none) -> PTS645SM43SMTR92; Manufacturer (none) -> C&K
- TX1, TX2, TX3, TX4: MPN (none) -> XL-1608UBC-04; Manufacturer (none) -> XINGLIGHT
- U1: MPN (none) -> RP2040; Manufacturer (none) -> Raspberry Pi
- U2: MPN (none) -> MAX-M10S-00B; Manufacturer (none) -> u-blox
- U3: MPN (none) -> MP2307DN-LF-Z; Manufacturer (none) -> Monolithic Power Systems (MPS)
- Y1: MPN (none) -> ABMM2-12.000MHZ-D1-T; Manufacturer (none) -> ABRACON
Connections:
- net +3.3V: now also C26.2, C27.2, C31.2, C32.1, JP2.1 (A), U4.12 (~{CS}), U4.5 (VDDIO), U4.8 (VDD)
- net +BATT: now also Q6.1 (S), Q6.2 (S), Q6.3 (S), Q8.1 (S), Q8.2 (S), Q8.3 (S)
- net GND: now also C26.1, C27.1, C31.1, C32.2, D3.1 (A1), JP2.3 (B), U4.6 (GND@6), U4.7 (GND@7)
- net I2C_SCL: now also U4.13 (SCL)
- net I2C_SDA: now also U4.14 (SDA)
- net at J9.1 (Pin_1), R64.1: now also Q6.5 (D)
- net at R58.1: now also Q8.4 (G)
- net at R62.1: now also Q6.4 (G)
- net at J10.1 (Pin_1), R60.1: now also Q8.5 (D)
- net at E22-400M22S1.21 (ANT), J11.1 (In): now also D3.2 (A2)
- new net: JP2.2 (C), U4.1 (SDO/SA0)
- no-connect marks 41 -> 40
Other:
- moved on the sheet: R17, R25
