File: ARC_PFC.kicad_sch (KiCad schematic)
At the start: 144 parts, among them IC1 TPS5430MDDAREP, IC4 TPS259531DSGR, IC5 BMP388, IC6 W25Q32JVSSIQ, J1 USB4216-03-A, J10 Conn_01x02, J11 Conn_Coaxial, J12 Conn_Coaxial, J2 BATTERY_CONN, J3 SWD_CONN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

Commit message: v2 fixes
Parts:
- R8: value 2.94k -> 3k
- SW1: value SW_Push -> RESET
- SW2: value SW_Push -> BOOT
Changed lines of the file:
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@@
 			)
 		)
-		(property "Value" "SW_Push"
+		(property "Value" "BOOT"
 			(at 490.22 149.86 0)
 			(show_name no)
@@
 			)
 		)
-		(property "Value" "2.94k"
-			(at 463.042 256.54 0)
+		(property "Value" "3k"
+			(at 465.328 256.286 0)
 			(show_name no)
 			(do_not_autoplace no)
@@
 			)
 		)
-		(property "Value" "SW_Push"
+		(property "Value" "RESET"
 			(at 45.72 237.49 0)
 			(show_name no)
