File: ARC_PFC.kicad_pcb (KiCad board)
At the start: 4 copper layers, 50 x 88.5 mm, 145 parts, among them IC1 TPS5430MDDAREP, IC4 TPS259531DSGR, IC5 BMP388, IC6 W25Q32JVSSIQ, J1 USB4216-03-A, J10 Conn_01x02, J11 Conn_Coaxial, J12 Conn_Coaxial, J2 BATTERY_CONN, J3 SWD_CONN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

Commit message: v2 fixes
Other:
- board text added: "BOOT"
- board text added: "RESET"
Changed lines of the file:
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@@
 			(outputformat 1)
 			(mirror no)
-			(drillshape 1)
+			(drillshape 0)
 			(scaleselection 1)
-			(outputdirectory "")
+			(outputdirectory "production/")
 		)
 	)
@@
 		)
 	)
+	(gr_line
+		(start 105 165.5)
+		(end 105 173)
+		(stroke
+			(width 0.08382)
+			(type solid)
+		)
+		(layer "B.SilkS")
+	)
+	(gr_line
+		(start 105 165.5)
+		(end 135 165.5)
+		(stroke
+			(width 0.08382)
+			(type solid)
+		)
+		(layer "B.SilkS")
+	)
+	(gr_line
+		(start 105 173)
+		(end 135 173)
+		(stroke
+			(width 0.08382)
+			(type solid)
+		)
+		(layer "B.SilkS")
+	)
+	(gr_line
+		(start 135 173)
+		(end 135 165.5)
+		(stroke
+			(width 0.08382)
+			(type solid)
+		)
+		(layer "B.SilkS")
+	)
 	(gr_arc
 		(start 95 89.5)
@@
 		(layer "Edge.Cuts")
 	)
-	(gr_text "SERVO"
-		(at 96.052866 107.437966 0)
-		(layer "F.SilkS")
-		(effects
-			(font
-				(size 1 1)
-				(thickness 0.1)
-			)
-			(justify left bottom)
-		)
-	)
-	(gr_text "SERVO"
-		(at 138.62 106.942442 0)
-		(layer "F.SilkS")
-		(effects
-			(font
-				(size 1 1)
-				(thickness 0.1)
-			)
-			(justify left bottom)
-		)
-	)
 	(gr_text "BATT"
 		(at 102.5 163 90)
@@
 		)
 	)
+	(gr_text "SERVO"
+		(at 96.052866 107.437966 0)
+		(layer "F.SilkS")
+		(effects
+			(font
+				(size 1 1)
+				(thickness 0.2)
+				(bold yes)
+			)
+			(justify left bottom)
+		)
+	)
 	(gr_text "2026"
 		(at 97.55 103.89 0)
@@
 		)
 	)
+	(gr_text "SERVO"
+		(at 138.62 106.942442 0)
+		(layer "F.SilkS")
+		(effects
+			(font
+				(size 1 1)
+				(thickness 0.2)
+				(bold yes)
+			)
+			(justify left bottom)
+		)
+	)
+	(gr_text "BOOT"
+		(at 130.5 135.5 0)
+		(layer "F.SilkS")
+		(effects
+			(font
+				(size 1.2 1.2)
+				(thickness 0.3)
+				(bold yes)
+			)
+			(justify left bottom)
+		)
+	)
+	(gr_text "RESET"
+		(at 130 150.5 270)
+		(layer "F.SilkS")
+		(effects
+			(font
+				(size 1.2 1.2)
+				(thickness 0.3)
+				(bold yes)
+			)
+			(justify left bottom)
+		)
+	)
 	(gr_text "RTU\nHPR"
 		(at 97.08 102.18 0)
@@
 	)
 	(via
-		(at 132.5 135.5)
+		(at 133.5 135.9)
 		(size 0.6)
 		(drill 0.3)
