File: _restore_backup_2026-06-27T18-31-22-950/ARC_PFC.kicad_pcb (KiCad board)
At the start: 4 copper layers, 50 x 88.5 mm, 145 parts, among them IC1 TPS5430MDDAREP, IC4 TPS259531DSGR, IC5 BMP388, IC6 W25Q32JVSSIQ, J1 USB4216-03-A, J10 Conn_01x02, J11 Conn_Coaxial, J12 Conn_Coaxial, J2 BATTERY_CONN, J3 SWD_CONN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

Commit message: v2 update
Parts:
- removed BT1: Battery_Cell, Battery:BatteryHolder_Seiko_MS621F
- removed D6, D7: D_Schottky, Diode_SMD:D_SOD-523
- removed D8: 1N4148W, Diode_SMD:D_SOD-123
- removed Q7: Q_NPN_BEC, Package_TO_SOT_SMD:SOT-23
- added Q1: 2N3904, Package_TO_SOT_SMD:SOT-23, F.Cu at (132.4, 171.8)
- C12: value 10nF -> 0.1nF
- C23: value 4.7nF -> 4.7uF
- C44, D5, R55: moved to F.Cu
- R8: value 2.94k -> 3.24k
- moved C44 64.2 mm to (76.9, 114.5)
- moved R55 63.4 mm to (77.0, 112.5), turned to 0 degrees
- moved D5 61.8 mm to (77.8, 108.2), turned to 0 degrees
Routing:
- net +5V: track 131.7 -> 62.9 mm, vias 11 -> 5
- net +3.3V: track 272.5 -> 244.1 mm, vias 14 -> 12
- net /5V_USB: track 38.2 -> 10.6 mm, vias 1 -> 0
- net /V_BCKUP: track 20.5 -> 0.00 mm, vias 1 -> 0
- net /5V_BATT: track 20.2 -> 9.94 mm, vias 2 -> 0
- net /3.3V_BS: track 8.07 -> 2.70 mm, vias 1 -> 0
- net Net-(D5-K): track 3.08 -> 0.00 mm
- net Net-(C30-+): track 33.3 -> 34.8 mm
- net GND: track 247.5 -> 246.1 mm, vias 57 -> 58
- net Net-(Q1-B): track 12.3 -> 13.4 mm
Other:
- board text added: "2025"
- board text removed: "2026"
