File: _restore_backup_2026-06-27T18-31-22-950/ARC_PFC.kicad_sch (KiCad schematic)
At the start: 144 parts, among them IC1 TPS5430MDDAREP, IC4 TPS259531DSGR, IC5 BMP388, IC6 W25Q32JVSSIQ, J1 USB4216-03-A, J10 Conn_01x02, J11 Conn_Coaxial, J12 Conn_Coaxial, J2 BATTERY_CONN, J3 SWD_CONN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

Commit message: v2 update
Parts:
- removed D6, D7: D_Schottky, Diode_SMD:D_SOD-523, symbol Device:D_Schottky
- removed D8: 1N4148W, Diode_SMD:D_SOD-123, symbol Device:D
- removed Q7: Q_NPN_BEC, Package_TO_SOT_SMD:SOT-23, symbol Transistor_BJT:Q_NPN_BEC
- added Q1: 2N3904, Package_TO_SOT_SMD:SOT-23, symbol Transistor_BJT:2N3904
- BT1: footprint Battery:BatteryHolder_Seiko_MS621F -> Battery:BatteryHolder_MPD_BC2003_1x2032
- C12: value 10nF -> 0.1nF
- C23: value 4.7nF -> 4.7uF
- R8: value 2.94k -> 3.24k
Connections:
- net GND: now also Q1.1 (E)
- net at R20.1: now also Q1.2 (B)
- net at BZ1.2 (-): now also Q1.3 (C)
Other:
- note removed: "5V SYSTEM"
- moved on the sheet: BZ1, C15, C16, C17, C18, C19, C39, C40, J10, J6, L1, L2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
